File: hw/picowater.kicad_pcb (KiCad board)
At the start: 2 copper layers, 98 x 56 mm, 47 parts, among them J1 +12V, J10 Batt TP, J13 RJ45, J14 RJ45, J15 RJ45, J2 Power In, J4 UART, J6 JST-PH2 Bat, J7 GPIO2, J9 5V TP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

Commit message: [case] adjust screw positions, minor tweaks
Parts:
- moved K1 2.90 mm to (127.8, 114.9)
- moved D3 2.90 mm to (124.3, 110.2)
- moved H1 1.41 mm to (58.5, 72.5)
- moved H2 1.41 mm to (147.5, 72.5)
- moved H3 1.41 mm to (58.5, 119.5)
- moved H4 1.41 mm to (147.5, 119.5)
Routing:
- net +12V: track 61.8 -> 59.2 mm
- net PUMP+12V: track 59.6 -> 58.2 mm
- net +5V: track 54.4 -> 53.2 mm
Changed lines of the file:
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@@
 	(footprint "MountingHole:MountingHole_4.3mm_M4"
 		(layer "F.Cu")
-		(at 148.5 120.5)
+		(at 147.5 119.5)
 		(descr "Mounting Hole 4.3mm, no annular, M4")
 		(tags "mounting hole 4.3mm no annular m4")
 		(property "Reference" "H4"
-			(at 0 -5.3 0)
+			(at -2.9 -5.35 0)
 			(layer "F.SilkS")
 			(effects
@@
 	(footprint "Diode_SMD:D_SOD-123"
 		(layer "F.Cu")
-		(at 127.24 110.2975 90)
+		(at 124.34 110.2475 90)
 		(descr "SOD-123")
 		(tags "SOD-123")
@@
 	(footprint "MountingHole:MountingHole_4.3mm_M4"
 		(layer "F.Cu")
-		(at 57.5 120.5)
+		(at 58.5 119.5)
 		(descr "Mounting Hole 4.3mm, no annular, M4")
 		(tags "mounting hole 4.3mm no annular m4")
@@
 	(footprint "Relay_THT:Relay_SPDT_Omron-G5Q-1"
 		(layer "F.Cu")
-		(at 130.71 114.98)
+		(at 127.81 114.93)
 		(descr "Relay SPDT Omron Serie G5Q, http://omronfs.omron.com/en_US/ecb/products/pdf/en-g5q.pdf")
 		(tags "Relay SPDT Omron Serie G5Q")
@@
 	(footprint "MountingHole:MountingHole_4.3mm_M4"
 		(layer "F.Cu")
-		(at 57.5 71.5)
+		(at 58.5 72.5)
 		(descr "Mounting Hole 4.3mm, no annular, M4")
 		(tags "mounting hole 4.3mm no annular m4")
@@
 	(footprint "MountingHole:MountingHole_4.3mm_M4"
 		(layer "F.Cu")
-		(at 148.5 71.5)
+		(at 147.5 72.5)
 		(descr "Mounting Hole 4.3mm, no annular, M4")
 		(tags "mounting hole 4.3mm no annular m4")
@@
 	)
 	(segment
-		(start 121.886008 92.59)
-		(end 107.83 92.59)
-		(width 0.5)
-		(layer "F.Cu")
-		(net 12)
-	)
-	(segment
-		(start 130.71 101.413992)
+		(start 107.83 92.59)
 		(end 121.886008 92.59)
 		(width 0.5)
@@
 	)
 	(segment
-		(start 130.71 107.36)
-		(end 128.5275 107.36)
+		(start 127.81 107.31)
+		(end 125.6275 107.31)
 		(width 0.7)
 		(layer "F.Cu")
@@
 	)
 	(segment
-		(start 128.5275 107.36)
-		(end 127.24 108.6475)
+		(start 127.81 98.513992)
+		(end 127.81 107.31)
+		(width 0.5)
+		(layer "F.Cu")
+		(net 12)
+	)
+	(segment
+		(start 125.6275 107.31)
+		(end 124.34 108.5975)
 		(width 0.7)
 		(layer "F.Cu")
@@
 	)
 	(segment
-		(start 130.71 107.36)
-		(end 130.71 101.413992)
+		(start 121.886008 92.59)
+		(end 127.81 98.513992)
 		(width 0.5)
 		(layer "F.Cu")
@@
 	)
 	(segment
-		(start 121.65 108.025)
-		(end 124.06 110.435)
+		(start 124.06 116.725)
+		(end 124.05 116.735)
 		(width 1)
 		(layer "F.Cu")
@@
 	)
 	(segment
-		(start 140.87 112.58)
-		(end 140.87 114.98)
+		(start 123.2785 107.8215)
+		(end 121.8535 107.8215)
+		(width 0.25)
+		(layer "F.Cu")
+		(net 13)
+	)
+	(segment
+		(start 137.97 112.53)
+		(end 137.97 114.93)
 		(width 1)
 		(layer "F.Cu")
@@
 	)
 	(segment
-		(start 123.24 94.9)
-		(end 124.63 96.29)
+		(start 124.63 106.47)
+		(end 123.2785 107.8215)
 		(width 0.25)
 		(layer "F.Cu")
@@
 	)
 	(segment
+		(start 121.65 109.32)
+		(end 121.65 108.025)
+		(width 1)
+		(layer "F.Cu")
+		(net 13)
+	)
+	(segment
 		(start 120.5 94.9)
 		(end 123.24 94.9)
@@
 	)
 	(segment
-		(start 124.06 116.725)
-		(end 124.05 116.735)
+		(start 120.65 110.32)
+		(end 121.65 109.32)
 		(width 1)
 		(layer "F.Cu")
@@
 	)
 	(segment
-		(start 121.65 108.025)
-		(end 118.625 105)
-		(width 1)
+		(start 124.63 96.29)
+		(end 124.63 106.47)
+		(width 0.25)
 		(layer "F.Cu")
 		(net 13)
 	)
 	(segment
-		(start 124.06 110.42)
-		(end 124.06 110.435)
-		(width 0.25)
+		(start 124.06 113.73)
+		(end 124.06 116.725)
+		(width 1)
 		(layer "F.Cu")
 		(net 13)
 	)
 	(segment
-		(start 124.06 110.435)
-		(end 124.06 116.725)
+		(start 120.65 110.32)
+		(end 124.06 113.73)
 		(width 1)
 		(layer "F.Cu")
@@
 	)
 	(segment
-		(start 124.63 96.29)
-		(end 124.63 109.85)
+		(start 121.8535 107.8215)
+		(end 121.65 108.025)
 		(width 0.25)
 		(layer "F.Cu")
@@
 	(segment
 		(start 115.65 110.32)
-		(end 138.61 110.32)
+		(end 135.66 110.32)
 		(width 1)
 		(layer "F.Cu")
@@
 	)
 	(segment
-		(start 138.61 110.32)
-		(end 140.87 112.58)
+		(start 115.51 110.18)
+		(end 115.65 110.32)
 		(width 1)
 		(layer "F.Cu")
@@
 	)
 	(segment
-		(start 124.63 109.85)
-		(end 124.06 110.42)
-		(width 0.25)
+		(start 135.71 110.27)
+		(end 137.97 112.53)
+		(width 1)
 		(layer "F.Cu")
 		(net 13)
 	)
 	(segment
-		(start 115.51 110.18)
-		(end 115.65 110.32)
+		(start 135.66 110.32)
+		(end 135.71 110.27)
 		(width 1)
 		(layer "F.Cu")
@@
 	)
 	(segment
+		(start 121.65 108.025)
+		(end 118.625 105)
+		(width 1)
+		(layer "F.Cu")
+		(net 13)
+	)
+	(segment
+		(start 123.24 94.9)
+		(end 124.63 96.29)
+		(width 0.25)
+		(layer "F.Cu")
+		(net 13)
+	)
+	(segment
 		(start 81.176 74.716)
 		(end 80 73.54)
@@
 	)
 	(segment
-		(start 127.24 111.95)
-		(end 130.71 115.42)
+		(start 124.34 111.9)
+		(end 127.81 115.37)
 		(width 0.7)
 		(layer "F.Cu")
@@
 	)
 	(segment
-		(start 127.24 111.9475)
-		(end 127.24 111.95)
+		(start 124.34 111.8975)
+		(end 124.34 111.9)
 		(width 0.7)
 		(layer "F.Cu")
@@
 	)
 	(segment
-		(start 130.71 115.42)
-		(end 130.71 117.0325)
+		(start 127.81 115.37)
+		(end 127.81 116.9825)
 		(width 0.7)
 		(layer "F.Cu")
@@
 	)
 	(segment
-		(start 148.49 114.52)
-		(end 137.66 103.69)
+		(start 137.66 107)
+		(end 137.66 99.13)
+		(width 0.5)
+		(layer "B.Cu")
+		(net 56)
+	)
+	(segment
+		(start 145.59 114.93)
+		(end 145.59 114.47)
 		(width 0.5)
 		(layer "B.Cu")
@@
 	)
 	(segment
-		(start 148.49 114.98)
-		(end 148.49 114.52)
+		(start 145.18 114.52)
+		(end 137.66 107)
 		(width 0.5)
 		(layer "B.Cu")
@@
 		(layer "B.Cu")
 		(net 56)
-	)
-	(segment
-		(start 137.66 103.69)
-		(end 137.66 99.13)
-		(width 0.5)
-		(layer "B.Cu")
-		(net 56)
